File: EG800AK-devboard.kicad_pcb (KiCad board)
At the start: 4 copper layers, 35 x 35 mm, 58 parts, among them J1 U.FL-R-SMT_10_, J2 MICROQTJ, J4 Conn_01x11_Pin, Q1 DTC143ZUAT106, Q2 DTC143ZUAT106, Q4 DTC143ZUAT106, Q5 DTC143ZUAT106, SW1 TS-1088-AR02016, U1 EG800KEULC-I03-SNNSA, U2 GPS1003

Commit message: carga
Parts:
- removed kibuzzard-6A62D0DC: G***, kibuzzard-6A62D0DC
- removed kibuzzard-6A62D141: G***, kibuzzard-6A62D141
- removed kibuzzard-6A62D254: G***, kibuzzard-6A62D254
- removed kibuzzard-6A62D2A4: G***, kibuzzard-6A62D2A4
- removed kibuzzard-6A62D2AF: G***, kibuzzard-6A62D2AF
- removed kibuzzard-6A62D2C7: G***, kibuzzard-6A62D2C7
- removed kibuzzard-6A62D2D6: G***, kibuzzard-6A62D2D6
- removed kibuzzard-6A62D322: G***, kibuzzard-6A62D322
- removed kibuzzard-6A62D32B: G***, kibuzzard-6A62D32B
- removed kibuzzard-6A642A22: G***, kibuzzard-6A642A22
- added kibuzzard-6A799EF0: G***, kibuzzard-6A799EF0, F.Cu at (212.9, 91.0)
- added kibuzzard-6A799EF5: G***, kibuzzard-6A799EF5, F.Cu at (212.9, 93.6)
- added kibuzzard-6A799F00: G***, kibuzzard-6A799F00, F.Cu at (212.9, 96.1)
- added kibuzzard-6A799F05: G***, kibuzzard-6A799F05, F.Cu at (212.8, 98.6)
- added kibuzzard-6A799F0B: G***, kibuzzard-6A799F0B, F.Cu at (212.9, 101.2)
- added kibuzzard-6A799F12: G***, kibuzzard-6A799F12, F.Cu at (212.9, 103.7)
- added kibuzzard-6A799F21: G***, kibuzzard-6A799F21, F.Cu at (212.8, 108.8)
- added kibuzzard-6A799F5E: G***, kibuzzard-6A799F5E, F.Cu at (212.8, 85.9)
- added kibuzzard-6A799F96: G***, kibuzzard-6A799F96, F.Cu at (212.8, 88.5)
- added kibuzzard-6A799FB4: G***, kibuzzard-6A799FB4, F.Cu at (212.8, 106.3)

Commit message: Eliminacion de GNSS, correcion final en nano_sim
Parts:
- removed U2: GPS1003, EasyEDA:ANT-SMD_L10.0-W3.0
- added kibuzzard-6AB957FC: G***, kibuzzard-6AB957FC, F.Cu at (230.2, 82.0)
- C17, C7, C8: value 470uF -> 100uF
Connections:
- C1 pad 2: Net-(C1-Pad2) -> Net-(NANO-SIM-0501A-P1-I/O)
- R4 pad 1: Net-(C1-Pad2) -> Net-(NANO-SIM-0501A-P1-I/O)
Routing:
- net Net-(NANO-SIM-0501A-P1-I/O): track 15.6 -> 29.6 mm
- net /GNSS: track 10.1 -> 0.00 mm
- net Net-(C1-Pad2): track 5.08 -> 0.00 mm
- net GND: track 44.7 -> 41.3 mm, vias 234 -> 207

Commit message: cambios finales
Parts:
- removed kibuzzard-6AB957FC: G***, kibuzzard-6AB957FC
- added kibuzzard-6AB97A40: G***, kibuzzard-6AB97A40, F.Cu at (227.3, 81.4)
- moved kibuzzard-6A62D453 3.54 mm to (215.3, 83.0)
- moved D6 3.37 mm to (215.3, 81.2)
- moved D7 3.37 mm to (210.0, 81.2)
- moved kibuzzard-6A62D44D 3.36 mm to (209.9, 82.9)
Routing:
- net GND: track 41.3 -> 24.0 mm, vias 207 -> 271
- net Net-(D6-K): track 2.00 -> 7.06 mm
- net Net-(D7-K): track 3.00 -> 6.23 mm
- net /DC 3.8v supply: track 98.8 -> 101.7 mm, vias 10 -> 11
- net /HOST.EG800K.PWRKEY: track 33.7 -> 36.5 mm
